Commit message: Add simulator-first scene and validated Ackermann Nav2 experiments

File: ros2_ws/src/gem_description/urdf/gem.urdf.xacro (robot description, xacro)
@@ -11,4 +11,9 @@
   <link name="base_footprint">
   </link>
+  <link name="base_rear_axle"/>
+  <joint name="base_rear_axle_joint" type="fixed">
+    <parent link="base_footprint"/><child link="base_rear_axle"/>
+    <origin xyz="-0.87 0 0" rpy="0 0 0"/>
+  </joint>
   <link name="base_link">
     <!--

Commit message: feat(tf): establish canonical E6 simulation frames

File: ros2_ws/src/gem_description/urdf/gem.urdf.xacro (robot description, xacro)
@@ -9,13 +9,14 @@
   <xacro:include filename="$(find gem_description)/urdf/materials.xacro" />
   <xacro:include filename="$(find gem_description)/urdf/macros.xacro" />
+  <!-- The simulation-only numeric transform registry is the single source for nominal frame values. -->
+  <xacro:property name="simulation_nominal_file" value="$(find gem_description)/config/e6/simulation_nominal_transforms.yaml"/>
+  <xacro:property name="simulation_nominal_config" value="${xacro.load_yaml(simulation_nominal_file)}"/>
+  <xacro:property name="sim_transforms" value="${simulation_nominal_config['transforms']}"/>
+  <xacro:property name="sim_supplemental_transforms" value="${simulation_nominal_config['simulation_scope']['supplemental_transforms']}"/>
   <!-- *************************** Base link below *************************** -->
-  <link name="base_footprint">
-  </link>
-  <link name="base_rear_axle"/>
-  <joint name="base_rear_axle_joint" type="fixed">
-    <parent link="base_footprint"/><child link="base_rear_axle"/>
-    <origin xyz="-0.87 0 0" rpy="0 0 0"/>
-  </joint>
-  <link name="base_link">
+  <!-- Canonical GEM e6 frame: rear-axle center projected to the ground. -->
+  <link name="base_link"/>
+  <!-- Preserve the inherited e2 body origin under the canonical rear-axle datum. -->
+  <link name="base_chassis_link">
     <!--
     <inertial>
@@ -56,8 +57,9 @@
     </collision>
   </link>
-  <joint name="base_link_joint" type="fixed">
-    <origin xyz="0 0 0.44" rpy="0 0 0"/>
-    <parent link="base_footprint"/>
-    <child link="base_link"/>
+  <joint name="base_chassis_joint" type="fixed">
+    <origin xyz="${sim_transforms['base_chassis_link']['translation_m'][0]} ${sim_transforms['base_chassis_link']['translation_m'][1]} ${sim_transforms['base_chassis_link']['translation_m'][2]}"
+            rpy="${sim_transforms['base_chassis_link']['rotation_rpy_rad'][0]} ${sim_transforms['base_chassis_link']['rotation_rpy_rad'][1]} ${sim_transforms['base_chassis_link']['rotation_rpy_rad'][2]}"/>
+    <parent link="base_link"/>
+    <child link="base_chassis_link"/>
   </joint>
   <!-- ******************************************* Fixed links below ******************************************* -->
@@ -90,5 +92,5 @@
   <joint name="chair_joint" type="fixed">
     <origin xyz="0.001 0 -0.02" rpy="0 0 0" />
-    <parent link="base_link" />
+    <parent link="base_chassis_link" />
     <child link="chair_link" />
     <axis xyz="0 0 0" />
@@ -122,5 +124,5 @@
   <joint name="door_joint" type="fixed">
     <origin xyz="0.001 0 -0.015" rpy="0 0 0" />
-    <parent link="base_link" />
+    <parent link="base_chassis_link" />
     <child link="door_link" />
     <axis xyz="0 0 0" />
@@ -152,9 +154,22 @@
     </collision>
   </link>
-  <joint name="top_rack_joint" type="fixed">
-    <origin xyz="-0.10172 0.6575 1.3921" rpy="1.5708 0 3.1416" />
+  <link name="top_sensor_rig_link">
+    <inertial>
+      <origin xyz="0 0 0" rpy="0 0 0"/>
+      <mass value="0.001"/>
+      <inertia ixx="1e-6" ixy="0" ixz="0" iyy="1e-6" iyz="0" izz="1e-6"/>
+    </inertial>
+  </link>
+  <joint name="top_sensor_rig_joint" type="fixed">
+    <origin xyz="${sim_transforms['top_sensor_rig_link']['translation_m'][0]} ${sim_transforms['top_sensor_rig_link']['translation_m'][1]} ${sim_transforms['top_sensor_rig_link']['translation_m'][2]}"
+            rpy="${sim_transforms['top_sensor_rig_link']['rotation_rpy_rad'][0]} ${sim_transforms['top_sensor_rig_link']['rotation_rpy_rad'][1]} ${sim_transforms['top_sensor_rig_link']['rotation_rpy_rad'][2]}" />
     <parent link="base_link" />
+    <child link="top_sensor_rig_link" />
+  </joint>
+  <!-- Retain the inherited rack mesh orientation while using a body-aligned rig datum. -->
+  <joint name="top_rack_visual_joint" type="fixed">
+    <origin xyz="0 0 0" rpy="1.5708 0 3.1416" />
+    <parent link="top_sensor_rig_link" />
     <child link="top_rack_link" />
-    <axis xyz="0 0 0" />
   </joint>
   <link name="front_rack_link">
@@ -186,5 +201,5 @@
   <joint name="front_rack_joint" type="fixed">
     <origin xyz="1.352 0 -0.30594" rpy="1.5708 0 1.5708" />
-    <parent link="base_link" />
+    <parent link="base_chassis_link" />
     <child link="front_rack_link" />
     <axis xyz="0 0 0" />
@@ -218,5 +233,5 @@
   <joint name="rear_rack_joint" type="fixed">
     <origin xyz="-1.302 0 -0.27168" rpy="1.5708 0 -1.5708" />
-    <parent link="base_link" />
+    <parent link="base_chassis_link" />
     <child link="rear_rack_link" />
     <axis xyz="0 0 0" />
@@ -250,5 +265,5 @@
   <joint name="front_right_head_light_joint" type="fixed">
     <origin xyz="0.755 -0.5 0.58706" rpy="0 0 0" />
-    <parent link="base_link" />
+    <parent link="base_chassis_link" />
     <child link="front_right_head_light_link" />
     <axis xyz="1 0 0" />
@@ -282,5 +297,5 @@
   <joint name="front_left_head_light_joint" type="fixed">
     <origin xyz="0.755 0.5 0.58706" rpy="0 0 0" />
-    <parent link="base_link" />
+    <parent link="base_chassis_link" />
     <child link="front_left_head_light_link" />
     <axis xyz="1 0 0" />
@@ -314,5 +329,5 @@
   <joint name="front_right_turn_light_joint" type="fixed">
     <origin xyz="0.765 -0.345 0.58706" rpy="0 0 0" />
-    <parent link="base_link" />
+    <parent link="base_chassis_link" />
     <child link="front_right_turn_light_link" />
     <axis xyz="1 0 0" />
@@ -346,5 +361,5 @@
   <joint name="front_left_turn_light_joint" type="fixed">
     <origin xyz="0.765 0.345 0.58706" rpy="0 0 0" />
-    <parent link="base_link" />
+    <parent link="base_chassis_link" />
     <child link="front_left_turn_light_link" />
     <axis xyz="1 0 0" />
@@ -378,5 +393,5 @@
   <joint name="rear_right_light_joint" type="fixed">
     <origin xyz="-1.195 -0.32 0.025063" rpy="0 0 0" />
-    <parent link="base_link" />
+    <parent link="base_chassis_link" />
     <child link="rear_right_light_link" />
     <axis xyz="1 0 0" />
@@ -410,5 +425,5 @@
   <joint name="rear_left_light_joint" type="fixed">
     <origin xyz="-1.195 0.32 0.025063" rpy="0 0 0" />
-    <parent link="base_link" />
+    <parent link="base_chassis_link" />
     <child link="rear_left_light_link" />
     <axis xyz="1 0 0" />
@@ -442,5 +457,5 @@
   <joint name="rear_left_stop_light_joint" type="fixed">
     <origin xyz="-1.195 0.38 0.24506" rpy="0 0 3.1416" />
-    <parent link="base_link" />
+    <parent link="base_chassis_link" />
     <child link="rear_left_stop_light_link" />
     <axis xyz="1 0 0" />
@@ -474,5 +489,5 @@
   <joint name="rear_right_stop_light_joint" type="fixed">
     <origin xyz="-1.195 -0.38 0.24506" rpy="0 0 3.1416" />
-    <parent link="base_link" />
+    <parent link="base_chassis_link" />
     <child link="rear_right_stop_light_link" />
     <axis xyz="1 0 0" />
@@ -506,5 +521,5 @@
   <joint name="right_blue_outer_joint" type="fixed">
     <origin xyz="0.002 -0.6745 0.23435" rpy="0 0 0" />
-    <parent link="base_link" />
+    <parent link="base_chassis_link" />
     <child link="right_blue_outer_link" />
     <axis xyz="0 0 0" />
@@ -538,5 +553,5 @@
   <joint name="right_AVL_joint" type="fixed">
     <origin xyz="-0.45 -0.7 0.08" rpy="0 0 0" />
-    <parent link="base_link" />
+    <parent link="base_chassis_link" />
     <child link="right_AVL_link" />
     <axis xyz="0 0 0" />
@@ -570,5 +585,5 @@
   <joint name="left_blue_outer_joint" type="fixed">
     <origin xyz="0.002 0.6645 0.23435" rpy="0 0 0" />
-    <parent link="base_link" />
+    <parent link="base_chassis_link" />
     <child link="left_blue_outer_link" />
     <axis xyz="0 0 0" />
@@ -602,5 +617,5 @@
   <joint name="left_AVL_joint" type="fixed">
     <origin xyz="-0.45 0.6 0.08" rpy="0 0 0" />
-    <parent link="base_link" />
+    <parent link="base_chassis_link" />
     <child link="left_AVL_link" />
     <axis xyz="0 0 0" />
@@ -634,5 +649,5 @@
   <joint name="right_antenna_joint" type="fixed">
     <origin xyz="-0.23472 -0.6125 1.5071" rpy="0 0 0" />
-    <parent link="base_link" />
+    <parent link="base_chassis_link" />
     <child link="right_antenna_link" />
     <axis xyz="0 0 1" />
@@ -666,5 +681,5 @@
   <joint name="left_antenna_joint" type="fixed">
     <origin xyz="-0.23472 0.6125 1.5071" rpy="0 0 0" />
-    <parent link="base_link" />
+    <parent link="base_chassis_link" />
     <child link="left_antenna_link" />
     <axis xyz="0 0 1" />
@@ -698,5 +713,5 @@
   <joint name="rear_left_emergency_button_joint" type="fixed">
     <origin xyz="-0.72012 0.6645 0.83815" rpy="0 0 0" />
-    <parent link="base_link" />
+    <parent link="base_chassis_link" />
     <child link="rear_left_emergency_button_link" />
     <axis xyz="0 1 0" />
@@ -730,5 +745,5 @@
   <joint name="rear_right_emergency_button_joint" type="fixed">
     <origin xyz="-0.72012 -0.6645 0.83815" rpy="0 0.57871 3.1416" />
-    <parent link="base_link" />
+    <parent link="base_chassis_link" />
     <child link="rear_right_emergency_button_link" />
     <axis xyz="0 1 0" />
@@ -762,5 +777,5 @@
   <joint name="front_left_emergency_button_joint" type="fixed">
     <origin xyz="1.1497 0.6645 0.20492" rpy="0 0 0" />
-    <parent link="base_link" />
+    <parent link="base_chassis_link" />
     <child link="front_left_emergency_button_link" />
     <axis xyz="0 1 0" />
@@ -794,5 +809,5 @@
   <joint name="front_right_emergency_button_joint" type="fixed">
     <origin xyz="1.1497 -0.6645 0.20492" rpy="0 0.57871 3.1416" />
-    <parent link="base_link" />
+    <parent link="base_chassis_link" />
     <child link="front_right_emergency_button_link" />
     <axis xyz="0 1 0" />
@@ -820,5 +835,5 @@
   <joint name="rear_light_bar_joint" type="fixed">
     <origin xyz="-0.64921 0 0.76944" rpy="-1.9138 0 1.5708" />
-    <parent link="base_link" />
+    <parent link="base_chassis_link" />
     <child link="rear_light_bar_link" />
     <axis xyz="0 0 0" />
@@ -847,5 +862,5 @@
   <joint name="front_camera_joint" type="fixed">
     <origin xyz="0.16 -0.11 1.1063" rpy="1.5708 0 -3.1416" />
-    <parent link="base_link" />
+    <parent link="base_chassis_link" />
     <child link="front_camera_link" />
     <axis xyz="0 0 0"/>
@@ -970,5 +985,5 @@
   </link>
   <joint name="left_steering_hinge_joint" type="revolute">
-    <parent link="base_link"/>
+    <parent link="base_chassis_link"/>
     <child link="left_steering_hinge_link"/>
     <origin xyz="0.88 0.6 -0.151" rpy="0 0 0"/>
@@ -977,5 +992,5 @@
   </joint>
   <joint name="right_steering_hinge_joint" type="revolute">
-    <parent link="base_link"/>
+    <parent link="base_chassis_link"/>
     <child link="right_steering_hinge_link"/>
     <origin xyz="0.88 -0.6 -0.151" rpy="0 0 0"/>
@@ -1005,5 +1020,5 @@
     <origin xyz="-0.87 0.6 -0.151" rpy="0 0 0"/>
     <axis xyz="0 1 0"/>
-    <parent link="base_link"/>
+    <parent link="base_chassis_link"/>
     <child link="rear_left_wheel_link"/>
     <limit effort="1000" velocity="100.0"/>
@@ -1012,5 +1027,5 @@
     <origin xyz="-0.87 -0.6 -0.151" rpy="0 0 0"/>
     <axis xyz="0 1 0"/>
-    <parent link="base_link"/>
+    <parent link="base_chassis_link"/>
     <child link="rear_right_wheel_link"/>
     <limit effort="1000" velocity="100.0"/>
@@ -1025,10 +1040,11 @@
   <!-- *********************************************** Sensors ************************************************ -->
   <!-- ************************* Front Camera ************************* -->
-  <joint name="gem_front_camera_joint" type="fixed">
-    <origin xyz="0.394 0 1.19" rpy="0 0 0"/>
+  <joint name="realsense_mount_joint" type="fixed">
+    <origin xyz="${sim_transforms['realsense_link']['translation_m'][0]} ${sim_transforms['realsense_link']['translation_m'][1]} ${sim_transforms['realsense_link']['translation_m'][2]}"
+            rpy="${sim_transforms['realsense_link']['rotation_rpy_rad'][0]} ${sim_transforms['realsense_link']['rotation_rpy_rad'][1]} ${sim_transforms['realsense_link']['rotation_rpy_rad'][2]}"/>
     <parent link="base_link"/>
-    <child link="stereo_camera_link"/>
-  </joint>
-  <link name="stereo_camera_link">
+    <child link="realsense_link"/>
+  </joint>
+  <link name="realsense_link">
     <collision>
       <origin xyz="0 0 0" rpy="0 0 0"/>
@@ -1050,11 +1066,18 @@
     </inertial>
   </link>
-  <link name="camera_front_optical_frame"/>
-  <joint name="camera_front_optical_joint" type="fixed">
-    <parent link="stereo_camera_link"/><child link="camera_front_optical_frame"/>
-    <origin xyz="0 0 0" rpy="${-PI/2} 0 ${-PI/2}"/>
-  </joint>
-  <!-- Camera Sensor for stereo_camera_link -->
-  <gazebo reference="stereo_camera_link">
+  <link name="realsense_color_optical_frame"/>
+  <joint name="realsense_color_optical_joint" type="fixed">
+    <parent link="realsense_link"/><child link="realsense_color_optical_frame"/>
+    <origin xyz="${sim_transforms['realsense_color_optical_frame']['translation_m'][0]} ${sim_transforms['realsense_color_optical_frame']['translation_m'][1]} ${sim_transforms['realsense_color_optical_frame']['translation_m'][2]}"
+            rpy="${sim_transforms['realsense_color_optical_frame']['rotation_rpy_rad'][0]} ${sim_transforms['realsense_color_optical_frame']['rotation_rpy_rad'][1]} ${sim_transforms['realsense_color_optical_frame']['rotation_rpy_rad'][2]}"/>
+  </joint>
+  <link name="realsense_depth_optical_frame"/>
+  <joint name="realsense_depth_optical_joint" type="fixed">
+    <parent link="realsense_link"/><child link="realsense_depth_optical_frame"/>
+    <origin xyz="${sim_transforms['realsense_depth_optical_frame']['translation_m'][0]} ${sim_transforms['realsense_depth_optical_frame']['translation_m'][1]} ${sim_transforms['realsense_depth_optical_frame']['translation_m'][2]}"
+            rpy="${sim_transforms['realsense_depth_optical_frame']['rotation_rpy_rad'][0]} ${sim_transforms['realsense_depth_optical_frame']['rotation_rpy_rad'][1]} ${sim_transforms['realsense_depth_optical_frame']['rotation_rpy_rad'][2]}"/>
+  </joint>
+  <!-- Generic Gazebo RGB-D stand-in using the canonical RealSense frame contract. -->
+  <gazebo reference="realsense_link">
     <sensor type="camera" name="front_camera">
       <update_rate>30.0</update_rate>
@@ -1078,5 +1101,5 @@
       </camera>
       <topic>camera/image_raw</topic>
-      <ignition_frame_id>camera_front_optical_frame</ignition_frame_id>
+      <ignition_frame_id>realsense_color_optical_frame</ignition_frame_id>
     </sensor>
     <xacro:if value="$(arg auxiliary_cameras)">
@@ -1098,9 +1121,10 @@
       <visualize>true</visualize>
       <topic>depth_camera/image_raw</topic>
+      <ignition_frame_id>realsense_depth_optical_frame</ignition_frame_id>
     </sensor>
     </xacro:if>
   </gazebo>
   <!-- IMU -->
-  <link name="IMU_link">
+  <link name="realsense_imu_frame">
     <collision>
       <origin xyz="0 0 0" rpy="0 0 0"/>
@@ -1125,11 +1149,12 @@
     </inertial>
   </link>
-  <joint name="IMU_joint" type="fixed">
-    <origin xyz="-0.246 0 0.05" rpy="0 0 -1.5708"/>
-    <parent link="base_link"/>
-    <child link="IMU_link"/>
-  </joint>
-  <!-- GPS -->
-  <link name="GPS_link">
+  <joint name="realsense_imu_joint" type="fixed">
+    <origin xyz="${sim_transforms['realsense_imu_frame']['translation_m'][0]} ${sim_transforms['realsense_imu_frame']['translation_m'][1]} ${sim_transforms['realsense_imu_frame']['translation_m'][2]}"
+            rpy="${sim_transforms['realsense_imu_frame']['rotation_rpy_rad'][0]} ${sim_transforms['realsense_imu_frame']['rotation_rpy_rad'][1]} ${sim_transforms['realsense_imu_frame']['rotation_rpy_rad'][2]}"/>
+    <parent link="realsense_link"/>
+    <child link="realsense_imu_frame"/>
+  </joint>
+  <!-- Retained legacy Gazebo NavSat fixture; not an E6 antenna phase-center model. -->
+  <link name="legacy_gnss_sim_link">
     <collision>
       <origin xyz="0 0 0" rpy="0 0 0"/>
@@ -1154,8 +1179,9 @@
     </inertial>
   </link>
-  <joint name="GPS_joint" type="fixed">
-    <origin xyz="-0.246 0 0.05" rpy="0 0 0"/>
-    <parent link="base_link"/>
-    <child link="GPS_link"/>
+  <joint name="legacy_gnss_sim_joint" type="fixed">
+    <origin xyz="${sim_supplemental_transforms['legacy_gnss_sim_link']['translation_m'][0]} ${sim_supplemental_transforms['legacy_gnss_sim_link']['translation_m'][1]} ${sim_supplemental_transforms['legacy_gnss_sim_link']['translation_m'][2]}"
+            rpy="${sim_supplemental_transforms['legacy_gnss_sim_link']['rotation_rpy_rad'][0]} ${sim_supplemental_transforms['legacy_gnss_sim_link']['rotation_rpy_rad'][1]} ${sim_supplemental_transforms['legacy_gnss_sim_link']['rotation_rpy_rad'][2]}"/>
+    <parent link="${sim_supplemental_transforms['legacy_gnss_sim_link']['parent']}"/>
+    <child link="legacy_gnss_sim_link"/>
   </joint>
   <!-- Front Sonar -->
@@ -1233,6 +1259,7 @@
   </link>
   <joint name="velodyne_joint" type="fixed">
-    <origin xyz="0.02 0.15 -0.6575" rpy="1.5708 0 3.1416" />
-    <parent link="top_rack_link"/>
+    <origin xyz="${sim_transforms['velodyne_link']['translation_m'][0]} ${sim_transforms['velodyne_link']['translation_m'][1]} ${sim_transforms['velodyne_link']['translation_m'][2]}"
+            rpy="${sim_transforms['velodyne_link']['rotation_rpy_rad'][0]} ${sim_transforms['velodyne_link']['rotation_rpy_rad'][1]} ${sim_transforms['velodyne_link']['rotation_rpy_rad'][2]}" />
+    <parent link="top_sensor_rig_link"/>
     <child link="velodyne_link"/>
   </joint>
@@ -1279,5 +1306,5 @@
       name="ignition::gazebo::systems::OdometryPublisher">
       <odom_frame>world</odom_frame>
-      <robot_base_frame>base_footprint</robot_base_frame>
+      <robot_base_frame>base_link</robot_base_frame>
       <odom_topic>/ground_truth/odometry</odom_topic>
       <dimensions>3</dimensions>
